File: kb_1/Mathias_ergo.sch (KiCad schematic (older format))
At the start: 38 parts, among them J1 Conn_01x04, J2 Conn_01x04, Q1 DMG3414U, Q2 DMG3414U, SW1 SW_Push_Dual, SW10 SW_Push_Dual, SW11 SW_Push_Dual, SW12 SW_Push_Dual, SW13 SW_Push_Dual, SW14 SW_Push_Dual, SW15 SW_Push_Dual, SW16 SW_Push_Dual, SW17 SW_Push_Dual, SW18 SW_Push_Dual, SW19 SW_Push_Dual, SW2 SW_Push_Dual, SW20 SW_Push_Dual, SW21 SW_Push_Dual, SW22 SW_Push_Dual, SW23 SW_Push_Dual, SW24 SW_Push_Dual, SW25 SW_Push_Dual, SW26 SW_Push_Dual, SW27 SW_Push_Dual, SW28 SW_Push_Dual, SW29 SW_SPST, SW3 SW_Push_Dual, SW30 SW_SPST, SW4 SW_Push_Dual, SW5 SW_Push_Dual, SW6 SW_Push_Dual, SW7 SW_Push_Dual, SW8 SW_Push_Dual, SW9 SW_Push_Dual

Commit message: Exported gerbers
Parts:
- MCU1, MCU2: symbol User:Core51822 -> Mathias_ergo-rescue:Core51822-User
Changed lines of the file:
@@
 Connection ~ 950  1600
 $Comp
-L User:Core51822 MCU1
+L Mathias_ergo-rescue:Core51822-User MCU1
 U 1 1 5E914475
 P 1400 2350
@@
 Connection ~ 950  5150
 $Comp
-L User:Core51822 MCU2
+L Mathias_ergo-rescue:Core51822-User MCU2
 U 1 1 5E97D228
 P 1400 5900
