File: kb_2/Mathias_ergo.sch (KiCad schematic (older format))
At the start: 35 parts, among them J1 Conn_01x04, J2 Conn_01x04, J3 Conn_02x02_Odd_Even, Q1 DMG3414U, Q2 DMG3414U, SW1 Kailh_choc, SW10 Kailh_choc, SW11 Kailh_choc, SW12 Kailh_choc, SW13 Kailh_choc, SW14 Kailh_choc, SW15 Kailh_choc, SW16 Kailh_choc, SW17 Kailh_choc, SW18 Kailh_choc, SW19 Kailh_choc, SW2 Kailh_choc, SW20 Kailh_choc, SW21 Kailh_choc, SW22 Kailh_choc, SW23 Kailh_choc, SW24 Kailh_choc, SW25 SW_SPST, SW26 SW_SPST, SW3 Kailh_choc, SW4 Kailh_choc, SW5 Kailh_choc, SW6 Kailh_choc, SW7 Kailh_choc, SW8 Kailh_choc, SW9 Kailh_choc

Commit message: added silkscreen
Signed-off-by: mojitas <47667093+Mojitas@users.noreply.github.com>
Parts:
- SW1, SW10, SW11, SW12, SW13, SW14, SW15, SW16, SW17, SW18, SW19, SW2, SW20, SW21, SW22, SW23, SW24, SW3, SW4, SW5, SW6, SW7, SW8, SW9: symbol User_Switch:SW_Push_Dual -> Mathias_ergo-rescue:SW_Push_Dual-User_Switch
Changed lines of the file:
@@
 NoConn ~ 950  7200
 $Comp
-L User_Switch:SW_Push_Dual SW17
+L Mathias_ergo-rescue:SW_Push_Dual-User_Switch SW17
 U 1 1 5EF82529
 P 6550 2600
@@
 $EndComp
 $Comp
-L User_Switch:SW_Push_Dual SW18
+L Mathias_ergo-rescue:SW_Push_Dual-User_Switch SW18
 U 1 1 5EF8A940
 P 7600 2600
@@
 $EndComp
 $Comp
-L User_Switch:SW_Push_Dual SW19
+L Mathias_ergo-rescue:SW_Push_Dual-User_Switch SW19
 U 1 1 5EF92AF6
 P 8700 2600
@@
 $EndComp
 $Comp
-L User_Switch:SW_Push_Dual SW22
+L Mathias_ergo-rescue:SW_Push_Dual-User_Switch SW22
 U 1 1 5EFABBE3
 P 6550 3150
@@
 	5500 3350 5650 3350
 $Comp
-L User_Switch:SW_Push_Dual SW21
+L Mathias_ergo-rescue:SW_Push_Dual-User_Switch SW21
 U 1 1 5EFC4FD1
 P 5300 3150
@@
 	5550 2800 5650 2800
 $Comp
-L User_Switch:SW_Push_Dual SW16
+L Mathias_ergo-rescue:SW_Push_Dual-User_Switch SW16
 U 1 1 5EF7A22A
 P 5350 2600
@@
 S23
 $Comp
-L User_Switch:SW_Push_Dual SW20
+L Mathias_ergo-rescue:SW_Push_Dual-User_Switch SW20
 U 1 1 5EF9B0F9
 P 9900 2600
@@
 S6
 $Comp
-L User_Switch:SW_Push_Dual SW23
+L Mathias_ergo-rescue:SW_Push_Dual-User_Switch SW23
 U 1 1 5EFB4459
 P 7600 3150
@@
 $EndComp
 $Comp
-L User_Switch:SW_Push_Dual SW24
+L Mathias_ergo-rescue:SW_Push_Dual-User_Switch SW24
 U 1 1 5EFBCB19
 P 8700 3150
@@
 Text Label 4400 5400 0    50   ~ 0
 Battery_switch_tht
-Text Notes 5250 4400 0    50   ~ 0
-This connection is for the THT battery holders
 Wire Wire Line
 	4400 5400 4400 5650
@@
 Connection ~ 8450 2800
 $Comp
-L User_Switch:SW_Push_Dual SW15
+L Mathias_ergo-rescue:SW_Push_Dual-User_Switch SW15
 U 1 1 5EF71D21
 P 9900 2050
@@
 $EndComp
 $Comp
-L User_Switch:SW_Push_Dual SW10
+L Mathias_ergo-rescue:SW_Push_Dual-User_Switch SW10
 U 1 1 5EF48A4E
 P 9900 1500
@@
 $EndComp
 $Comp
-L User_Switch:SW_Push_Dual SW5
+L Mathias_ergo-rescue:SW_Push_Dual-User_Switch SW5
 U 1 1 5EF1F1CF
 P 9900 950
@@
 	5550 950  5550 1150
 $Comp
-L User_Switch:SW_Push_Dual SW1
+L Mathias_ergo-rescue:SW_Push_Dual-User_Switch SW1
 U 1 1 5EF0544A
 P 5350 950
@@
 $EndComp
 $Comp
-L User_Switch:SW_Push_Dual SW6
+L Mathias_ergo-rescue:SW_Push_Dual-User_Switch SW6
 U 1 1 5EF2775E
 P 5350 1500
@@
 $EndComp
 $Comp
-L User_Switch:SW_Push_Dual SW11
+L Mathias_ergo-rescue:SW_Push_Dual-User_Switch SW11
 U 1 1 5EF50F21
 P 5350 2050
@@
 S29
 $Comp
-L User_Switch:SW_Push_Dual SW14
+L Mathias_ergo-rescue:SW_Push_Dual-User_Switch SW14
 U 1 1 5EF69911
 P 8700 2050
@@
 $EndComp
 $Comp
-L User_Switch:SW_Push_Dual SW13
+L Mathias_ergo-rescue:SW_Push_Dual-User_Switch SW13
 U 1 1 5EF615D4
 P 7600 2050
@@
 $EndComp
 $Comp
-L User_Switch:SW_Push_Dual SW12
+L Mathias_ergo-rescue:SW_Push_Dual-User_Switch SW12
 U 1 1 5EF59304
 P 6550 2050
@@
 $EndComp
 $Comp
-L User_Switch:SW_Push_Dual SW9
+L Mathias_ergo-rescue:SW_Push_Dual-User_Switch SW9
 U 1 1 5EF404DF
 P 8700 1500
@@
 $EndComp
 $Comp
-L User_Switch:SW_Push_Dual SW8
+L Mathias_ergo-rescue:SW_Push_Dual-User_Switch SW8
 U 1 1 5EF38059
 P 7600 1500
@@
 $EndComp
 $Comp
-L User_Switch:SW_Push_Dual SW7
+L Mathias_ergo-rescue:SW_Push_Dual-User_Switch SW7
 U 1 1 5EF2FD1C
 P 6550 1500
@@
 $EndComp
 $Comp
-L User_Switch:SW_Push_Dual SW4
+L Mathias_ergo-rescue:SW_Push_Dual-User_Switch SW4
 U 1 1 5EF16D8E
 P 8700 950
@@
 $EndComp
 $Comp
-L User_Switch:SW_Push_Dual SW3
+L Mathias_ergo-rescue:SW_Push_Dual-User_Switch SW3
 U 1 1 5EF0E9E9
 P 7600 950
@@
 $EndComp
 $Comp
-L User_Switch:SW_Push_Dual SW2
+L Mathias_ergo-rescue:SW_Push_Dual-User_Switch SW2
 U 1 1 5EF06446
 P 6550 950
@@
 Text Notes 2750 3650 0    50   ~ 0
 Connectors for testing if the unsused\ngnd plane can be used for debouncing.
+Text Notes 5250 4400 0    50   ~ 0
+This connection is for the THT battery holders
 $EndSCHEMATC

Commit message: Send to factory version
Parts:
- added H101, H102, H103, H104, H105, H106: MountingHole, MountingHole:MountingHole_2.2mm_M2_Pad_Via, symbol Mechanical:MountingHole
Changed lines of the file:
@@
 Text Notes 5250 4400 0    50   ~ 0
 This connection is for the THT battery holders
+$Comp
+L Mechanical:MountingHole H101
+U 1 1 6022320A
+P 6250 6600
+F 0 "H101" H 6350 6646 50  0000 L CNN
+F 1 "MountingHole" H 6350 6555 50  0000 L CNN
+F 2 "MountingHole:MountingHole_2.2mm_M2_Pad_Via" H 6250 6600 50  0001 C CNN
+F 3 "~" H 6250 6600 50  0001 C CNN
+	1    6250 6600
+	1    0    0    -1
+$EndComp
+$Comp
+L Mechanical:MountingHole H102
+U 1 1 60223856
+P 6250 6750
+F 0 "H102" H 6350 6796 50  0000 L CNN
+F 1 "MountingHole" H 6350 6705 50  0000 L CNN
+F 2 "MountingHole:MountingHole_2.2mm_M2_Pad_Via" H 6250 6750 50  0001 C CNN
+F 3 "~" H 6250 6750 50  0001 C CNN
+	1    6250 6750
+	1    0    0    -1
+$EndComp
+$Comp
+L Mechanical:MountingHole H103
+U 1 1 60223A37
+P 6250 6900
+F 0 "H103" H 6350 6946 50  0000 L CNN
+F 1 "MountingHole" H 6350 6855 50  0000 L CNN
+F 2 "MountingHole:MountingHole_2.2mm_M2_Pad_Via" H 6250 6900 50  0001 C CNN
+F 3 "~" H 6250 6900 50  0001 C CNN
+	1    6250 6900
+	1    0    0    -1
+$EndComp
+$Comp
+L Mechanical:MountingHole H104
+U 1 1 60223B94
+P 6250 7050
+F 0 "H104" H 6350 7096 50  0000 L CNN
+F 1 "MountingHole" H 6350 7005 50  0000 L CNN
+F 2 "MountingHole:MountingHole_2.2mm_M2_Pad_Via" H 6250 7050 50  0001 C CNN
+F 3 "~" H 6250 7050 50  0001 C CNN
+	1    6250 7050
+	1    0    0    -1
+$EndComp
+$Comp
+L Mechanical:MountingHole H105
+U 1 1 60223D44
+P 6250 7200
+F 0 "H105" H 6350 7246 50  0000 L CNN
+F 1 "MountingHole" H 6350 7155 50  0000 L CNN
+F 2 "MountingHole:MountingHole_2.2mm_M2_Pad_Via" H 6250 7200 50  0001 C CNN
+F 3 "~" H 6250 7200 50  0001 C CNN
+	1    6250 7200
+	1    0    0    -1
+$EndComp
+$Comp
+L Mechanical:MountingHole H106
+U 1 1 60223F19
+P 6250 7350
+F 0 "H106" H 6350 7396 50  0000 L CNN
+F 1 "MountingHole" H 6350 7305 50  0000 L CNN
+F 2 "MountingHole:MountingHole_2.2mm_M2_Pad_Via" H 6250 7350 50  0001 C CNN
+F 3 "~" H 6250 7350 50  0001 C CNN
+	1    6250 7350
+	1    0    0    -1
+$EndComp
 $EndSCHEMATC

Commit message: Exported gerbers
Parts:
- H101, H102, H103, H104, H105, H106: footprint MountingHole:MountingHole_2.2mm_M2_Pad_Via -> MountingHole:MountingHole_2.2mm_M2_Pad
Changed lines of the file:
@@
 F 0 "H101" H 6350 6646 50  0000 L CNN
 F 1 "MountingHole" H 6350 6555 50  0000 L CNN
-F 2 "MountingHole:MountingHole_2.2mm_M2_Pad_Via" H 6250 6600 50  0001 C CNN
+F 2 "MountingHole:MountingHole_2.2mm_M2_Pad" H 6250 6600 50  0001 C CNN
 F 3 "~" H 6250 6600 50  0001 C CNN
 	1    6250 6600
@@
 F 0 "H102" H 6350 6796 50  0000 L CNN
 F 1 "MountingHole" H 6350 6705 50  0000 L CNN
-F 2 "MountingHole:MountingHole_2.2mm_M2_Pad_Via" H 6250 6750 50  0001 C CNN
+F 2 "MountingHole:MountingHole_2.2mm_M2_Pad" H 6250 6750 50  0001 C CNN
 F 3 "~" H 6250 6750 50  0001 C CNN
 	1    6250 6750
@@
 F 0 "H103" H 6350 6946 50  0000 L CNN
 F 1 "MountingHole" H 6350 6855 50  0000 L CNN
-F 2 "MountingHole:MountingHole_2.2mm_M2_Pad_Via" H 6250 6900 50  0001 C CNN
+F 2 "MountingHole:MountingHole_2.2mm_M2_Pad" H 6250 6900 50  0001 C CNN
 F 3 "~" H 6250 6900 50  0001 C CNN
 	1    6250 6900
@@
 F 0 "H104" H 6350 7096 50  0000 L CNN
 F 1 "MountingHole" H 6350 7005 50  0000 L CNN
-F 2 "MountingHole:MountingHole_2.2mm_M2_Pad_Via" H 6250 7050 50  0001 C CNN
+F 2 "MountingHole:MountingHole_2.2mm_M2_Pad" H 6250 7050 50  0001 C CNN
 F 3 "~" H 6250 7050 50  0001 C CNN
 	1    6250 7050
@@
 F 0 "H105" H 6350 7246 50  0000 L CNN
 F 1 "MountingHole" H 6350 7155 50  0000 L CNN
-F 2 "MountingHole:MountingHole_2.2mm_M2_Pad_Via" H 6250 7200 50  0001 C CNN
+F 2 "MountingHole:MountingHole_2.2mm_M2_Pad" H 6250 7200 50  0001 C CNN
 F 3 "~" H 6250 7200 50  0001 C CNN
 	1    6250 7200
@@
 F 0 "H106" H 6350 7396 50  0000 L CNN
 F 1 "MountingHole" H 6350 7305 50  0000 L CNN
-F 2 "MountingHole:MountingHole_2.2mm_M2_Pad_Via" H 6250 7350 50  0001 C CNN
+F 2 "MountingHole:MountingHole_2.2mm_M2_Pad" H 6250 7350 50  0001 C CNN
 F 3 "~" H 6250 7350 50  0001 C CNN
 	1    6250 7350
