File: kb_2/Mathias_ergo.kicad_pcb (KiCad board)
At the start: 2 copper layers, 187.6 x 123.8 mm, 41 parts, among them J1 Conn_01x04, J2 Conn_01x04, J3 Conn_02x02_Odd_Even, Q1 DMG3414U, Q2 DMG3414U, SW1 Kailh_choc, SW10 Kailh_choc, SW11 Kailh_choc, SW12 Kailh_choc, SW13 Kailh_choc, SW14 Kailh_choc, SW15 Kailh_choc, SW16 Kailh_choc, SW17 Kailh_choc, SW18 Kailh_choc, SW19 Kailh_choc, SW2 Kailh_choc, SW20 Kailh_choc, SW21 Kailh_choc, SW22 Kailh_choc, SW23 Kailh_choc, SW24 Kailh_choc, SW25 SW_SPST, SW26 SW_SPST, SW3 Kailh_choc, SW4 Kailh_choc, SW5 Kailh_choc, SW6 Kailh_choc, SW7 Kailh_choc, SW8 Kailh_choc, SW9 Kailh_choc

Commit message: added silkscreen
Signed-off-by: mojitas <47667093+Mojitas@users.noreply.github.com>
Parts:
- removed the REF** at (121.3, 66.1)
- removed the REF** at (216.1, 70.1)
- removed the REF** at (157.6, 120.7)
- removed the REF** at (217.1, 136.9)
- removed the REF** at (90.0, 172.5)
- removed the REF** at (52.0, 127.6)
- added REF**: MountingHole_2.2mm_M2_Pad_Via, MountingHole:MountingHole_2.2mm_M2_Pad_Via, F.Cu at (216.1, 70.1)
- added REF**: MountingHole_2.2mm_M2_Pad_Via, MountingHole:MountingHole_2.2mm_M2_Pad_Via, F.Cu at (121.3, 66.1)
- added REF**: MountingHole_2.2mm_M2_Pad_Via, MountingHole:MountingHole_2.2mm_M2_Pad_Via, F.Cu at (217.1, 136.9)
- added REF**: MountingHole_2.2mm_M2_Pad_Via, MountingHole:MountingHole_2.2mm_M2_Pad_Via, F.Cu at (157.6, 120.7)
- added REF**: MountingHole_2.2mm_M2_Pad_Via, MountingHole:MountingHole_2.2mm_M2_Pad_Via, F.Cu at (89.6, 171.3)
- added REF**: MountingHole_2.2mm_M2_Pad_Via, MountingHole:MountingHole_2.2mm_M2_Pad_Via, F.Cu at (52.1, 127.6)
Other:
- board text added: "Botkeeb rev 1.0"

Commit message: Design rules check
Signed-off-by: mojitas <47667093+Mojitas@users.noreply.github.com>
Other:
- net class Default: clearance 0.2032 -> 0.2; trace_width 0.2032 -> 0.2
- rule trace_clearance: 0.2032 -> 0.2
- rule trace_min: 0.127 -> 0.2
Changed lines of the file:
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@@
   )
   (page A4)
+  (title_block
+    (title Botkeeb)
+    (date 2020-11-13)
+    (rev 1.0)
+    (company "Mojitas upcoming company")
+  )
   (layers
     (0 F.Cu signal)
@@
   )
   (setup
-    (last_trace_width 0.2032)
+    (last_trace_width 0.2)
     (user_trace_width 0.25)
-    (trace_clearance 0.2032)
+    (trace_clearance 0.2)
     (zone_clearance 0.508)
     (zone_45_only no)
-    (trace_min 0.127)
+    (trace_min 0.2)
     (via_size 0.8)
     (via_drill 0.4)
@@
   (net 49 /Battery_switch_tht)
   (net_class Default "This is the default net class."
-    (clearance 0.2032)
-    (trace_width 0.2032)
+    (clearance 0.2)
+    (trace_width 0.2)
     (via_dia 0.8)
     (via_drill 0.4)

Commit message: New outline
Fixed the board outline,
thumb buttons positions,
battery footprint,
gnd pours
Parts:
- removed the REF** at (217.1, 136.9)
- removed the REF** at (157.6, 120.7)
- removed the REF** at (89.6, 171.3)
- added REF**: M2_Mount, MountingHole:MountingHole_2.2mm_M2_Pad_Via, F.Cu at (215.4, 133.4)
- added REF**: M2_Mount, MountingHole:MountingHole_2.2mm_M2_Pad_Via, F.Cu at (158.1, 120.5)
- added REF**: M2_Mount, MountingHole:MountingHole_2.2mm_M2_Pad_Via, F.Cu at (100.2, 163.2)
- REF** (x2): value MountingHole_2.2mm_M2_Pad_Via -> M2_Mount
- REF**: value MountingHole_2.2mm_M2_Pad_Via -> M2_mount
- SW25, SW26: footprint User_Keyboard:PCM12SMTR -> User_Keyboard:PCM12SMTR_via_pads
- moved REF** 29.7 mm to (79.5, 116.2)
- moved SW15 3.51 mm to (80.2, 139.7), turned to 40.5 degrees
- moved SW3 3.03 mm to (92.6, 154.2), turned to 40.5 degrees
- moved MCU1 2.79 mm to (92.3, 108.9)
- moved MCU2 2.79 mm to (92.3, 108.9)
- moved SW13 2.48 mm to (100.9, 125.8), turned to 27 degrees
- moved SW4 2.17 mm to (109.6, 142.8), turned to 27 degrees
- moved SW23 1.39 mm to (128.7, 135.7), turned to 13.5 degrees
- moved J1 1.01 mm to (63.6, 128.8), turned to 130.5 degrees
- moved SW18 1.00 mm to (149.0, 133.3)
- moved J2 0.85 mm to (69.4, 123.8), turned to 130.5 degrees
Routing:
- net /S14: track 66.6 -> 73.0 mm
- net /S29: track 110.5 -> 116.4 mm
- net /S20: track 103.1 -> 108.8 mm
- net /S6: track 95.4 -> 90.0 mm
- net /S30: track 174.7 -> 169.4 mm
- net /S11: track 135.0 -> 129.8 mm
- net /S12: track 211.4 -> 206.2 mm
- net /S5: track 285.6 -> 280.5 mm
- net /S22: track 248.4 -> 243.4 mm
- net /S3: track 150.8 -> 155.6 mm
- net /S17: track 190.8 -> 194.5 mm
- net /S26: track 182.5 -> 179.0 mm
- net /S19: track 230.9 -> 234.3 mm
- net /S23: track 271.1 -> 274.0 mm
- net /S9: track 260.1 -> 257.3 mm
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Other:
- board size 187.6 x 123.8 mm -> 174.4 x 119.5 mm
- board text added: "Botkeeb rev 1.1"
- board text removed: "Botkeeb rev 1.0"

Commit message: Send to factory version
Parts:
- removed REF** (x5): M2_Mount, MountingHole:MountingHole_2.2mm_M2_Pad_Via
- removed REF**: M2_mount, MountingHole:MountingHole_2.2mm_M2_Pad_Via
- added H101: MountingHole, MountingHole:MountingHole_2.2mm_M2_Pad_Via, F.Cu at (100.2, 163.2)
- added H102: MountingHole, MountingHole:MountingHole_2.2mm_M2_Pad_Via, F.Cu at (79.5, 116.2)
- added H103: MountingHole, MountingHole:MountingHole_2.2mm_M2_Pad_Via, F.Cu at (158.1, 120.5)
- added H104: MountingHole, MountingHole:MountingHole_2.2mm_M2_Pad_Via, F.Cu at (121.0, 65.9)
- added H105: MountingHole, MountingHole:MountingHole_2.2mm_M2_Pad_Via, F.Cu at (215.4, 133.4)
- added H106: MountingHole, MountingHole:MountingHole_2.2mm_M2_Pad_Via, F.Cu at (216.2, 70.9)
- SW25, SW26: footprint User_Keyboard:PCM12SMTR_via_pads -> User_Keyboard:PCM12SMTR
- moved SW25 48.4 mm to (210.1, 139.8), turned to 28 degrees
- moved SW26 48.4 mm to (210.1, 139.8), turned to 208 degrees
- moved Q1 38.3 mm to (197.2, 142.9), turned to 270 degrees
- moved Q2 38.3 mm to (197.2, 142.9), turned to 270 degrees
- moved J3 7.72 mm to (195.9, 130.7)
- moved BT1 3.77 mm to (175.8, 135.3)
- moved BT2 3.77 mm to (175.8, 135.3)
Routing:
- net /Battery_switch_tht: track 53.2 -> 68.6 mm, vias 0 -> 1
- net Net-(BT2-Pad2): track 17.9 -> 26.5 mm
- net Net-(BT1-Pad2): track 18.2 -> 26.4 mm
- net VCC2: track 245.2 -> 237.4 mm
- net VCC1: track 237.1 -> 233.0 mm
Other:
- board text added: "Off"
- board text added: "On"

Commit message: Exported gerbers
Parts:
- H101, H102, H103, H104, H105, H106: footprint MountingHole:MountingHole_2.2mm_M2_Pad_Via -> MountingHole:MountingHole_2.2mm_M2_Pad
- moved J1 31.5 mm to (94.3, 136.0)
- moved J2 31.5 mm to (100.1, 131.1)
- moved Q1 31.5 mm to (227.8, 150.2)
- moved Q2 31.5 mm to (227.8, 150.2)
- moved H101 31.5 mm to (130.9, 170.5)
- moved H105 31.5 mm to (246.0, 140.6)
- moved SW18 31.5 mm to (179.7, 140.6)
- moved SW5 31.5 mm to (246.9, 127.6)
- moved H106 31.5 mm to (246.9, 78.2)
- moved J3 31.5 mm to (226.6, 138.0)
- moved SW12 31.5 mm to (246.9, 91.5)
- moved SW24 31.5 mm to (151.6, 86.5)
- moved SW8 31.5 mm to (208.8, 99.5)
- moved SW25 31.5 mm to (240.8, 147.1)
- moved SW26 31.5 mm to (240.8, 147.1)
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Routing:
- net /Battery_switch_tht: track 68.6 -> 35.8 mm
- net /S29: track 116.4 -> 112.6 mm
- net /S3: track 155.6 -> 152.0 mm
- net /S19: track 234.3 -> 230.7 mm
- net /S23: track 274.0 -> 270.5 mm
- net /S17: track 194.5 -> 191.3 mm
- net /S14: track 73.0 -> 70.7 mm
- net /S1: track 52.2 -> 53.7 mm
- net /S2: track 93.1 -> 94.5 mm
- net /S18: track 147.3 -> 146.2 mm
- net /SWCLK2: track 29.4 -> 30.3 mm
- net VCC2: track 237.4 -> 238.3 mm
- net /S24: track 80.6 -> 81.4 mm
- net /SWCLK1: track 39.0 -> 39.8 mm
- net /S16: track 115.9 -> 116.7 mm
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Other:
- net class Default: clearance 0.2 -> 0.127; trace_width 0.2 -> 0.127; via_dia 0.8 -> 0.6; via_drill 0.4 -> 0.3
- rule pad_to_mask_clearance: 0.05 -> 0
- rule solder_mask_min_width: 0.2 -> 0.12
- rule trace_clearance: 0.2 -> 0.127
- rule trace_min: 0.2 -> 0.127
- rule via_min_drill: 0.2 -> 0.3
- rule via_min_size: 0.45 -> 0.6
- board text added: "JLCJLCJLCJLC"

Commit message: Added more clearances between traces
Parts:
- moved H102 386.3 mm to (12.9, 497.3)
- moved SW23 383.7 mm to (66.6, 515.4)
- moved SW7 383.7 mm to (58.8, 494.9)
- moved SW8 383.7 mm to (116.0, 471.9)
- moved H103 383.7 mm to (95.9, 500.2)
- moved SW19 383.7 mm to (96.9, 484.9)
- moved SW16 383.7 mm to (116.0, 453.8)
- moved BT1 383.7 mm to (113.7, 514.9)
- moved BT2 383.7 mm to (113.7, 514.9)
- moved SW3 383.7 mm to (30.5, 533.8)
- moved SW14 383.7 mm to (77.9, 489.9)
- moved SW24 383.7 mm to (58.8, 458.8)
- moved SW2 383.7 mm to (77.9, 453.8)
- moved SW12 383.7 mm to (154.1, 463.8)
- moved SW21 383.7 mm to (58.8, 476.9)
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Routing:
- net /S20: track 108.9 -> 101.8 mm
- net /S5: track 280.5 -> 276.9 mm
- net VCC2: track 238.3 -> 241.5 mm
- net /S22: track 243.4 -> 240.8 mm
- net /S1: track 53.7 -> 51.6 mm
- net /SWCLK1: track 39.8 -> 41.6 mm
- net /SWDIO1: track 38.2 -> 39.8 mm
- net /S14: track 70.7 -> 69.2 mm
- net /S18: track 146.2 -> 144.9 mm
- net /S4: track 67.2 -> 66.0 mm
- net /S16: track 116.7 -> 115.5 mm
- net /S29: track 112.6 -> 111.4 mm
- net /S17: track 191.3 -> 192.4 mm
- net /S9: track 257.3 -> 256.2 mm
- net /SWDIO2: track 34.9 -> 35.9 mm
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Other:
- net class Default: clearance 0.127 -> 0.254
- net class JLC added: clearance 0.254, trace_width 0.2, via_dia 0.6, via_drill 0.3
- rule trace_clearance: 0.127 -> 0.254

Commit message: added last
Signed-off-by: Mathias <47667093+Mojitas@users.noreply.github.com>
Parts:
- moved Q1 181.2 mm to (-30.4, 448.9)
- moved Q2 181.2 mm to (-30.4, 448.9)
- moved SW25 143.3 mm to (34.7, 431.7)
- moved SW26 143.3 mm to (34.7, 431.7)
- moved J3 126.6 mm to (22.8, 449.4)
- moved BT2 112.5 mm to (10.0, 471.3), turned to 220.5 degrees
- moved BT1 111.8 mm to (10.6, 471.6), turned to 40.5 degrees
- moved J1 88.2 mm to (74.1, 458.2), turned to 90 degrees
- moved J2 87.1 mm to (81.7, 458.2), turned to 90 degrees
- moved H105 17.5 mm to (136.8, 518.9)
- moved MCU2 14.6 mm to (38.5, 476.5), turned to 180 degrees
- moved MCU1 14.6 mm to (38.4, 476.5), turned to 0 degrees
- moved H102 13.7 mm to (10.2, 510.8)
Routing:
- net VCC2: track 241.5 -> 0.00 mm
- net VCC1: track 233.2 -> 0.00 mm
- net /S6: track 90.8 -> 25.0 mm
- net /S11: track 130.3 -> 68.4 mm
- net /S30: track 169.6 -> 109.3 mm
- net /S12: track 205.4 -> 146.0 mm
- net /S22: track 240.8 -> 184.8 mm
- net /S5: track 276.9 -> 224.3 mm
- net /S4: track 66.0 -> 15.9 mm
- net /S25: track 102.0 -> 58.3 mm
- net /SWCLK1: track 41.6 -> 0.00 mm
- net /S7: track 142.9 -> 101.4 mm
- net /SWDIO1: track 39.8 -> 0.00 mm
- net /S26: track 178.8 -> 140.6 mm
- net /SWDIO2: track 35.9 -> 0.00 mm
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Other:
- board text removed: "Debounce right"
