File: kb_2/Mathias_ergo.kicad_pcb (KiCad board)
At the start: 2 copper layers, 174.4 x 119.5 mm, 41 parts, among them J1 Conn_01x04, J2 Conn_01x04, J3 Conn_02x02_Odd_Even, Q1 DMG3414U, Q2 DMG3414U, SW1 Kailh_choc, SW10 Kailh_choc, SW11 Kailh_choc, SW12 Kailh_choc, SW13 Kailh_choc, SW14 Kailh_choc, SW15 Kailh_choc, SW16 Kailh_choc, SW17 Kailh_choc, SW18 Kailh_choc, SW19 Kailh_choc, SW2 Kailh_choc, SW20 Kailh_choc, SW21 Kailh_choc, SW22 Kailh_choc, SW23 Kailh_choc, SW24 Kailh_choc, SW25 SW_SPST, SW26 SW_SPST, SW3 Kailh_choc, SW4 Kailh_choc, SW5 Kailh_choc, SW6 Kailh_choc, SW7 Kailh_choc, SW8 Kailh_choc, SW9 Kailh_choc

Commit message: pushing before wipe
Signed-off-by: Mathias Strand <47667093+Mojitas@users.noreply.github.com>
Parts:
- removed J3: Conn_02x02_Odd_Even, Connector_PinHeader_2.54mm:PinHeader_2x02_P2.54mm_Vertical
- removed SW15, SW18: Kailh_choc, User_Keyboard:Kailh_low_profile
- added D1: CQY99, Diode_SMD:D_0603_1608Metric, F.Cu at (89.8, 93.2)
- added D2: CQY99, Diode_SMD:D_0603_1608Metric, B.Cu at (89.8, 93.2)
- added H105: MountingHole, MountingHole:MountingHole_2.2mm_M2_Pad, F.Cu at (171.0, 61.8)
- added R1: R_Small, Resistor_SMD:R_0603_1608Metric, F.Cu at (89.8, 90.1)
- added R2: R_Small, Resistor_SMD:R_0603_1608Metric, B.Cu at (89.8, 90.1)
- added S1: 482020514001, MDU_solar:SW_482020514001, F.Cu at (82.2, 139.6)
- added S2: 482020514001, MDU_solar:SW_482020514001, B.Cu at (82.2, 139.6)
- moved H102 407.4 mm to (96.3, 112.6)
- moved H101 404.5 mm to (99.4, 143.1)
- moved H103 392.2 mm to (160.2, 113.3)
- moved H105 389.9 mm to (198.4, 134.0)
- moved SW19 387.9 mm to (160.3, 102.2)
- moved SW1 387.9 mm to (160.3, 66.1)
- moved SW17 387.9 mm to (160.3, 84.1)
- moved MCU1 387.9 mm to (99.9, 93.6)
- moved MCU2 387.8 mm to (99.9, 93.6)
- moved SW8 386.9 mm to (179.3, 90.1)
- moved SW16 386.9 mm to (179.3, 72.1)
- moved SW14 386.9 mm to (141.2, 108.2)
- moved SW20 386.9 mm to (179.3, 108.2)
- moved SW9 386.9 mm to (141.2, 90.1)
- moved SW2 386.9 mm to (141.2, 72.1)
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Connections:
- MCU1 pad 0: /S2 -> /S1
- MCU1 pad 1: /S18 -> /S2
- MCU1 pad 21: Net-(MCU1-Pad21) -> /D1
- MCU1 pad 22: Net-(MCU1-Pad22) -> unconnected-(MCU1-Pad22)
- MCU1 pad 23: Net-(MCU1-Pad23) -> unconnected-(MCU1-Pad23)
- MCU1 pad 24: Net-(MCU1-Pad24) -> unconnected-(MCU1-Pad24)
- MCU1 pad 25: Net-(MCU1-Pad25) -> /S24
- MCU1 pad 28: /S24 -> /S8
- MCU1 pad 29: /S16 -> /S10
- MCU1 pad 30: /S1 -> /S16
- MCU1 pad 35: Net-(MCU1-Pad35) -> unconnected-(MCU1-Pad35)
- MCU1 pad 36: Net-(MCU1-Pad36) -> unconnected-(MCU1-Pad36)
- MCU2 pad 11: /S18 -> /S2
- MCU2 pad 12: /S2 -> /S1
- MCU2 pad 13: /S1 -> /S16
- MCU2 pad 14: /S16 -> /S8
- MCU2 pad 15: /S24 -> /S10
- MCU2 pad 16: Net-(MCU2-Pad16) -> /S24
- MCU2 pad 17: Net-(MCU2-Pad17) -> unconnected-(MCU2-Pad17)
- MCU2 pad 18: Net-(MCU2-Pad18) -> unconnected-(MCU2-Pad18)
- MCU2 pad 19: Net-(MCU2-Pad19) -> unconnected-(MCU2-Pad19)
- MCU2 pad 20: Net-(MCU2-Pad20) -> /D2
- MCU2 pad 35: Net-(MCU2-Pad35) -> unconnected-(MCU2-Pad35)
- MCU2 pad 36: Net-(MCU2-Pad36) -> unconnected-(MCU2-Pad36)
- SW25 pad : (no net) -> VCC1
- SW26 pad : (no net) -> VCC2
Routing:
- net /S18: track 121.9 -> 0.00 mm
- net /S8: track 0.00 -> 107.0 mm
- net /S10: track 0.00 -> 106.9 mm
- net VCC2: track 0.00 -> 82.9 mm
- net VCC1: track 0.00 -> 70.3 mm
- net /S9: track 223.4 -> 271.9 mm
- net /S13: track 181.6 -> 225.5 mm
- net /S5: track 224.3 -> 268.2 mm
- net /S16: track 83.1 -> 126.5 mm
- net /S24: track 49.9 -> 92.5 mm
- net /S1: track 39.2 -> 81.3 mm
- net /S22: track 184.8 -> 222.9 mm
- net /S2: track 78.7 -> 115.3 mm
- net /SWCLK1: track 0.00 -> 33.7 mm
- net /S17: track 165.6 -> 195.9 mm
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Other:
- board size 174.4 x 119.5 mm -> 172.3 x 112.1 mm
- net class Default removed
- net class JLC removed
- board text added: "Le Bob"
- board text removed: "Botkeeb rev 1.1"
- board text removed: "Debounce left"
- board text removed: "Off"
- board text removed: "On"
